File: bluetooth-tracker.kicad_pcb (KiCad board)
At the start: 4 copper layers, 35 x 35 mm, 25 parts, among them J1 CONN4PROG, Q1 FDV301N_G, U1 NRF51822-QFAA-T_G

Commit message: Commiting finished design files.
Other:
- board text added: "0.20 MM 0.20 MM 0.20 MM 0.20 MM"
- board text added: "0.20 MM 0.20 MM 0.20 MM 0.20 MM 0.25 MM"
- board text added: "0.8 MM +/- 0.1 MM"
- board text added: "B-STAGE"
- board text added: "BOT LAYER"
- board text added: "IN1 LAYER"
- board text added: "IN2 LAYER"
- board text added: "TOP LAYER"
- board text removed: ".063 +/- .005"
- board text removed: "10 MILS 10 MILS 7.5 MILS 125 MILS"
- board text removed: "10 MILS 25 MILS 0.2 MM 25 MILS 15 MILS"
- board text removed: "B-STAGE (.013 REF)"
- board text removed: "INT2 LAYER"
- board text removed: "TOP LAYER (VOLTAGE/RTN SIGNAL TRACES)"
