File: bluetooth-tracker.sch (KiCad schematic (older format))
At the start: 25 parts, among them J1 CONN4PROG, Q1 FDV301N_G, U1 NRF51822-QFAA-T_G

Commit message: Commiting finished design files.
Changed lines of the file:
@@
 U 1 1 5E9F68AC
 P 7950 4900
-F 0 "GN1" H 7950 5567 50  0000 C CNN
-F 1 "BAL-NRF01D3" H 7650 4199 50  0000 L BNN
+F 0 "GN1" H 7950 5450 50  0000 C CNN
+F 1 "BAL-NRF01D3" H 7700 4300 50  0000 L BNN
 F 2 "global-library:FCBGA-5N" H 7950 4900 50  0001 L BNN
 F 3 "https://www.st.com/content/ccc/resource/technical/document/datasheet/88/54/7c/fd/6d/9c/46/74/DM00055606.pdf/files/DM00055606.pdf/jcr:content/translations/en.DM00055606.pdf" H 7950 4900 50  0001 L BNN
@@
 F 3 "http://infocenter.nordicsemi.com/pdf/nRF51822_PB_v2.5.pdf" H 5050 4300 60  0001 L CNN
 F 4 "1490-1024-ND" H 5050 4400 60  0001 L CNN "Digi-Key_PN"
-F 5 "NRF51822-QFAA-T" H 5050 4500 60  0001 L CNN "MPN"
+F 5 "NRF51822-QFAA-T" H 3800 1800 60  0000 L CNN "MPN"
 F 6 "RF/IF and RFID" H 5050 4600 60  0001 L CNN "Category"
 F 7 "RF Transceiver ICs" H 5050 4700 60  0001 L CNN "Family"
@@
 P 1300 3300
 F 0 "BAT1" H 1418 3353 60  0000 L CNN
-F 1 "CR2032_CLIP2" H 1250 3150 60  0000 R CNN
+F 1 "CR2032_CLIP2" H 1250 3150 60  0001 R CNN
 F 2 "global-library:CR2032_CLIP2" H 1500 3500 60  0001 L CNN
 F 3 "https://www.memoryprotectiondevices.com/datasheets/BK-912-datasheet.pdf" V 1500 3600 60  0001 L CNN
@@
 U 1 1 5E9DEFCE
 P 9450 3850
-F 0 "L3" V 9645 3850 50  0000 C CNN
-F 1 "3.3nH" H 9475 3750 50  0000 L CNN
+F 0 "L3" V 9550 3850 50  0000 C CNN
+F 1 "3.3nH" V 9400 3750 50  0000 L CNN
 F 2 "Inductor_SMD:L_0402_1005Metric" H 9488 3700 50  0001 C CNN
 F 3 "https://search.murata.co.jp/Ceramy/image/img/P02/JELF243C-0007.pdf" H 9450 3850 50  0001 C CNN
@@
 P 1850 1200
 F 0 "J1" H 1822 1174 50  0000 R CNN
-F 1 "CONN4PROG" H 1850 900 50  0000 C CNN
+F 1 "CONN4PROG" H 1850 900 50  0001 C CNN
 F 2 "global-library:CONN4PROG" H 1850 1200 50  0001 C CNN
 F 3 "~" H 1850 1200 50  0001 C CNN
